Commit message: bug hunt

File: robbie/urdf/mantis_gripper.xacro (robot description, xacro)
@@ -48,5 +48,5 @@
    <visual>
       <geometry>
-        <mesh filename="package://robbiemesh/claw_3_l.stl" scale="${M_SCALE} ${M_SCALE} ${M_SCALE}"/>
+        <mesh filename="package://robbie/mesh/claw_3_l.stl" scale="${M_SCALE} ${M_SCALE} ${M_SCALE}"/>
       </geometry>
          <xacro:White/>
